File: Hardware/han_to_wifi_board/han_to_wifi_board.kicad_sch (KiCad schematic)
At the start: 36 parts, among them IC1 MIC2779L-2YM5_TR, IC3 MAX17644AATE+, J1 RJLSE4118101, J3 Conn_01x05_Male, SW1 RESET, SW2 PRGRM, U1 ESP-12F, U3 NCN5150

Commit message: Changes after first bringup
Parts:
- L3: footprint Inductor_SMD:L_Vishay_IHLP-2020 -> IHLP2020BZER5R6M11:L_Vishay_IHLP-2020
- SW1, SW2: footprint Button_Switch_SMD:SW_SPST_EVQP2 -> EVQP2:EVQP2; symbol Switch:SW_Push_Dual -> Switch:SW_Push_Dual_x2
Connections:
- net GND: no longer IC3.4 (MODE/SYNC)
- net ~{HAN}: now also U3.7 (TXI); no longer U3.13 (RXI)
- net ~{RST}: now also R1.1, U1.3 (EN); no longer IC3.8 (~{RESET})
- no-connect marks 24 -> 22
Other:
- note removed: "RS232"
